File: PSMPS/PSMPS.kicad_sch (KiCad schematic)
At the start: 49 parts, among them J2 Conn_01x06, J4 USB_C_Receptacle, J5 Conn_01x04, Q7 MMBT5551L, Q8 MMBT5551L, SW1 MCU_RESET, SW3 MCU_RESET, SW3 RotaryEncoder_Switch, U1 ESP32-S3-WROOM-1, U11 LM324A, U12 STM32F030C8Tx, U4 SRV05-4, U5 MCP6002-xSN, U9 CJ431

Commit message: g
Connections:
- net ESP_BOOT: now also U12.44 (BOOT0)
Changed lines of the file:
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@@
+    (stroke (width 0) (type default))
+  )
+  (wire (pts (xy 187.325 52.705) (xy 197.485 52.705))
     (stroke (width 0) (type default))
   )
@@
     (effects (font (size 1.27 1.27)) (justify right bottom))
   )
+  (label "ESP_BOOT" (at 187.325 52.705 0) (fields_autoplaced)
+    (effects (font (size 1.27 1.27)) (justify left bottom))
+  )
   (label "GPIO_16" (at 143.51 59.69 180) (fields_autoplaced)

Commit message: g
Parts:
- removed C37: 1n, Capacitor_SMD:C_1206_3216Metric, symbol Device:C_Small
- removed J4: USB_C_Receptacle, Connector_USB:USB_C_Receptacle_HRO_TYPE-C-31-M-12, symbol Connector:USB_C_Receptacle
- removed R32, R33: 5k1, Resistor_SMD:R_0402_1005Metric, symbol Device:R_Small
- added C14 (x2), C15 (x2): 10u, Capacitor_SMD:C_0603_1608Metric, symbol Device:C_Small
- added J2: USB_A, Connector_USB:USB_A_Molex_67643_Horizontal, symbol Connector:USB_A
- added R36: 10k, Resistor_SMD:R_0603_1608Metric_Pad0.98x0.95mm_HandSolder, symbol Device:R_Small
- added SW4: SW_SPDT, symbol Switch:SW_SPDT
- added SW5: SW_DIP_x08, symbol Switch:SW_DIP_x08
Connections:
- net +3V3: now also C14.1, C14.1, C15.1, C15.1, SW4.3 (C)
- net D+: now also J2.3 (D+)
- net D-: now also J2.2 (D-)
- net ESP_BOOT: no longer U12.44 (BOOT0)
- net ESP_EN: now also U12.7 (NRST)
- net GND: now also C14.2, C14.2, C15.2, C15.2, J2.4 (GND), SW4.1 (A)
- net VBUS: now also J2.1 (VBUS)
- new net: R36.1, SW4.2 (B)
- new net BOOT0: R36.2, U12.44 (BOOT0)
- no-connect marks 19 -> 10
Other:
- moved on the sheet: C14, C15
